File: Schematics/I_O.kicad_sch (KiCad schematic)
At the start: 12 parts, among them J1 1989751, J9 1989764, Q4 XP263N1001TR-G, U4 SP3220ECA-L, U5 SP485CN-L_TR

Commit message: Layout complete of the two PCBs
Parts:
- removed J9: 1989764, footprints:1989764, symbol mylib_sym:1989764
- added J9: 85513-5113, footprints:855135113, symbol mylib_sym:85513-5113
- R33: value 470R -> 220R
Connections:
- net +3.6V: now also J9.7 (White/Brown), J9.8 (Brown)
- net GND: now also J9.9 (Shield)
- net A: now reaches U5.6 (A)
- net A: now also R33.2, J9.1 (White/Orange,(Tx+)); no longer R33.1
- net B: now reaches U5.7 (B)
- net B: now also R33.1, J9.2 (Orange,(Tx–)); no longer R33.2
- net at Q4.3 (D): now also J9.5 (White/Blue), J9.6 (Green,(Rx–))
Other:
- moved on the sheet: C19, Q4, R33, U5
