File: Schematics/Sensor Board/Sensor Board.kicad_pcb (KiCad board)
At the start: 2 copper layers, 57 x 42 mm, 42 parts, among them J1 UJ20-C-H-G-SMT-P16-TR, J2 Conn_01x05_Pin, J3 1989764, J4 1989764, J5 1989764, J6 1989764, U1 NCP115ASN330T2G, U2 AP3012KTR-G1, U3 CH340N, U4 STM32C011F6P6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

Commit message: Layout complete of the two PCBs
Parts:
- C4, C5, C6, C7, C8, D3, L2, R6, R7, R8, R9, U2, U4, U5: moved to B.Cu
- J5, J6: value 1989764 -> 85513-5113; footprint footprints:1989764 -> footprints:855135113
- R1: value 44.2 -> 44.2K
- R11: value 470R -> 120R
- moved J5 31.1 mm to (136.5, 109.1), turned to 180 degrees
- moved R8 28.7 mm to (129.3, 77.2), turned to 180 degrees
- moved R5 27.8 mm to (148.8, 80.9)
- moved J4 26.1 mm to (125.9, 79.2), turned to 0 degrees
- moved C7 17.3 mm to (138.0, 99.0), turned to 180 degrees
- moved C5 17.1 mm to (137.9, 100.8), turned to 180 degrees
- moved LED1 16.9 mm to (126.6, 102.5)
- moved R11 16.3 mm to (132.4, 89.5), turned to 0 degrees
- moved J2 15.7 mm to (132.3, 86.7)
- moved JP1 15.6 mm to (170.8, 94.5), turned to 180 degrees
- moved JP2 15.1 mm to (128.8, 91.3)
- moved R10 13.7 mm to (168.2, 92.8), turned to 90 degrees
- moved TP2 12.3 mm to (126.6, 96.1)
- moved TP3 11.6 mm to (123.7, 96.0)
- moved TP1 11.2 mm to (124.5, 87.6)
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Connections:
- net Net-(JP2-A) renamed /B
- J5 pad 1: +3.6V -> /A
- J5 pad 3: Net-(U5-B) -> GND
- J6 pad 1: +3.6V -> /A
- J6 pad 3: Net-(U5-B) -> GND
- R11 pad 2: Net-(U5-B) -> /A
- U5 pad 7: Net-(U5-B) -> /A
Routing:
- net Net-(J2-Pin_4): track 58.1 -> 133.4 mm, vias 5 -> 3
- net GND: track 50.9 -> 115.8 mm, vias 29 -> 28
- net Net-(U5-B): track 57.3 -> 0.00 mm, vias 2 -> 0
- net +3.6V: track 125.2 -> 69.2 mm, vias 2 -> 1
- net /RS485_DE: track 44.9 -> 0.00 mm, vias 2 -> 0
- net /A: track 0.00 -> 28.2 mm, vias 0 -> 1
- net /ANV_IN: track 30.2 -> 56.7 mm, vias 2 -> 4
- net Net-(U4-PA8): track 10.6 -> 33.1 mm, vias 1 -> 2
- net /RS485_RO: track 7.78 -> 29.0 mm
- net +12V: track 25.2 -> 46.0 mm
- net +3.3V: track 12.2 -> 32.8 mm, vias 5 -> 6
- net Net-(J2-Pin_3): track 19.7 -> 4.74 mm
- net /B: track 52.1 -> 38.1 mm, vias 3 -> 2
- net Net-(J2-Pin_2): track 19.0 -> 6.55 mm, vias 0 -> 1
- net /~{RS485_RE}: track 31.8 -> 20.4 mm, vias 2 -> 0
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Other:
- board text added: "Prog."
- board text removed: "+"
- board text removed: "A"
- board text removed: "B"
- board text removed: "Programming"

Commit message: Final release 1.1
Parts:
- C1, C3, C4, C5, C6, C7, C8: footprint SparkFun-Capacitor:C_0603_1608Metric -> Capacitor_SMD:C_0603_1608Metric
- D3: value SMF05CT2G -> SOT65P210X110-6N
- moved TP1 15.0 mm to (123.5, 102.6)
- moved U4 9.00 mm to (137.2, 102.2)
- moved C8 8.38 mm to (155.8, 101.7), turned to 90 degrees
- moved C5 8.10 mm to (145.0, 104.7), turned to -90 degrees
- moved U5 8.02 mm to (149.7, 100.8)
- moved C7 7.61 mm to (143.1, 104.7), turned to -90 degrees
- moved R11 4.47 mm to (128.4, 91.5), turned to -90 degrees
- moved R10 4.27 mm to (166.7, 88.8)
- moved R8 4.00 mm to (129.3, 81.2)
- moved JP2 3.52 mm to (127.8, 87.9), turned to -90 degrees
- moved LED1 3.49 mm to (126.6, 106.0)
- moved TP4 2.66 mm to (126.5, 101.5)
- moved TP2 2.52 mm to (126.3, 98.6)
- moved R2 2.50 mm to (163.1, 88.4)
- moved JP1 2.50 mm to (169.3, 92.5)
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Routing:
- net Net-(J2-Pin_4): track 133.4 -> 33.7 mm, vias 3 -> 0
- net /~{RS485_RE}: track 20.4 -> 48.0 mm, vias 0 -> 2
- net GND: track 115.8 -> 88.8 mm, vias 28 -> 22
- net /RS485_DE: track 0.00 -> 24.3 mm, vias 0 -> 2
- net /ANV_IN: track 56.7 -> 35.5 mm, vias 4 -> 0
- net Net-(U4-PA8): track 33.1 -> 12.0 mm, vias 2 -> 1
- net Net-(D3-CATHODE_5): track 17.4 -> 34.5 mm, vias 4 -> 0
- net Net-(D3-CATHODE_2): track 30.5 -> 45.5 mm
- net +12V: track 46.0 -> 31.9 mm, vias 2 -> 1
- net +3.3V: track 32.8 -> 45.8 mm, vias 6 -> 7
- net Net-(U4-PA4): track 0.00 -> 12.7 mm, vias 0 -> 1
- net /A: track 28.2 -> 40.7 mm, vias 1 -> 3
- net Net-(JP1-B): track 31.7 -> 22.0 mm
- net Net-(J2-Pin_3): track 4.74 -> 13.4 mm
- net Net-(J2-Pin_2): track 6.55 -> 14.6 mm, vias 1 -> 0
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Other:
- board text added: "Dat"
- board text added: "Gnd"
- board text added: "Sensor Board V1.1 13-Mar-26"
- board text removed: "+Vin"
- board text removed: "-"
- board text removed: "D"
- board text removed: "Data"
