File: Schematics/Sensor Board/Sensor Board.kicad_sch (KiCad schematic)
At the start: 42 parts, among them J1 UJ20-C-H-G-SMT-P16-TR, J2 Conn_01x05_Pin, J3 1989764, J4 1989764, J5 85513-5113, J6 85513-5113, U1 NCP115ASN330T2G, U2 AP3012KTR-G1, U3 CH340N, U4 STM32C011F6P6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

Commit message: Layout complete of the two PCBs
Connections:
- net GND: now also J5.4 (Blue), J5.5 (White/Blue)
Other:
- moved on the sheet: C8, R10, TP4, U5

Commit message: Final release 1.1
Parts:
- C4: footprint SparkFun-Capacitor:C_0603_1608Metric -> Capacitor_SMD:C_0603_1608Metric
